File: TimerS.kicad_pcb (KiCad board)
At the start: 2 copper layers, 140 x 65 mm, 65 parts, among them J1 Power, SW1 Start/Stop, SW2 Reset, U1 74LS90, U11 74LS90, U12 74LS47, U14 NA555P, U15 NA555P, U2 74LS47, U4 L7805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

Commit message: Production
Parts:
- added RV1: R_Potentiometer, Potentiometer_THT:Potentiometer_Piher_PT-6-V_Vertical, F.Cu at (124.8, 60.1)
- moved C2 71.2 mm to (139.5, 29.9)
- moved C3 71.2 mm to (134.7, 67.0)
- moved C4 71.2 mm to (134.7, 63.0)
- moved J1 71.2 mm to (149.5, 21.9)
- moved R28 71.2 mm to (81.1, 40.8)
- moved R29 71.2 mm to (83.6, 40.8)
- moved R9 71.2 mm to (134.9, 74.7)
- moved REF** 71.2 mm to (147.5, 59.9)
- moved SW1 71.2 mm to (150.8, 47.1)
- moved SW2 71.2 mm to (150.8, 75.1)
- moved U14 71.2 mm to (123.2, 74.7)
- moved U15 71.2 mm to (126.3, 41.1)
- moved U3 71.2 mm to (28.0, 23.2)
- moved U4 71.2 mm to (130.1, 24.5)
- moved C1 71.2 mm to (125.5, 29.9)
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Connections:
- R31 pad 2: Net-(U14-DIS) -> Net-(R31-Pad2)
Routing:
- net Net-(U14-DIS): track 6.43 -> 17.6 mm
- net +5V: track 581.9 -> 576.1 mm
- net Net-(U14-THR): track 25.8 -> 28.7 mm
- net Net-(R31-Pad2): track 0.00 -> 2.84 mm
- net GND: track 422.9 -> 424.3 mm
Other:
- board text added: "SAIDHAN ELECTRONICS"
- board text removed: "SAID ELECTRONICS"
