File: TimerS.kicad_sch (KiCad schematic)
At the start: 21 parts, among them J1 Power, SW1 Start/Stop, SW2 Reset, U14 NA555P, U15 NA555P, U4 L7805

Commit message: Production
Parts:
- added RV1: R_Potentiometer, Potentiometer_THT:Potentiometer_Piher_PT-6-V_Vertical, symbol Device:R_Potentiometer
Connections:
- net at R32.1, U14.7 (DIS): now also RV1.2, RV1.3; no longer R31.2
- new net: R31.2, RV1.1
Other:
- moved on the sheet: R31
Changed lines of the file:
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@@
   (junction (at 208.28 44.45) (diameter 0) (color 0 0 0 0)
   )
+  (junction (at 170.18 81.28) (diameter 0) (color 0 0 0 0)
+  )
   (junction (at 93.98 78.74) (diameter 0) (color 0 0 0 0)
   )
-  (junction (at 134.62 67.31) (diameter 0) (color 0 0 0 0)
-  )
   (junction (at 30.48 58.42) (diameter 0) (color 0 0 0 0)
   )
@@
   (junction (at 152.4 88.9) (diameter 0) (color 0 0 0 0)
   )
+  (junction (at 134.62 55.88) (diameter 0) (color 0 0 0 0)
+  )
   (junction (at 215.9 44.45) (diameter 0) (color 0 0 0 0)
   )
@@
     (stroke (width 0) (type default))
   )
+  (wire (pts (xy 134.62 50.8) (xy 134.62 55.88))
+    (stroke (width 0) (type default))
+  )
   (wire (pts (xy 255.27 95.25) (xy 255.27 83.82))
     (stroke (width 0) (type default))
@@
     (stroke (width 0) (type default))
   )
-  (wire (pts (xy 161.29 67.31) (xy 134.62 67.31))
-    (stroke (width 0) (type default))
-  )
   (wire (pts (xy 121.92 78.74) (xy 118.11 78.74))
     (stroke (width 0) (type default))
@@
     (stroke (width 0) (type default))
   )
+  (wire (pts (xy 170.18 76.2) (xy 170.18 81.28))
+    (stroke (width 0) (type default))
+  )
   (wire (pts (xy 87.63 93.98) (xy 93.98 93.98))
     (stroke (width 0) (type default))
@@
     (stroke (width 0) (type default))
   )
+  (wire (pts (xy 134.62 55.88) (xy 161.29 55.88))
+    (stroke (width 0) (type default))
+  )
   (wire (pts (xy 67.31 30.48) (xy 67.31 31.75))
     (stroke (width 0) (type default))
@@
     (stroke (width 0) (type default))
   )
+  (wire (pts (xy 161.29 81.28) (xy 161.29 80.01))
+    (stroke (width 0) (type default))
+  )
   (wire (pts (xy 118.11 78.74) (xy 118.11 69.85))
     (stroke (width 0) (type default))
@@
     (stroke (width 0) (type default))
   )
+  (wire (pts (xy 161.29 64.77) (xy 161.29 72.39))
+    (stroke (width 0) (type default))
+  )
   (wire (pts (xy 215.9 118.11) (xy 227.33 118.11))
     (stroke (width 0) (type default))
@@
     (stroke (width 0) (type default))
   )
-  (wire (pts (xy 134.62 64.77) (xy 134.62 67.31))
-    (stroke (width 0) (type default))
-  )
   (wire (pts (xy 72.39 93.98) (xy 72.39 88.9))
     (stroke (width 0) (type default))
@@
     (stroke (width 0) (type default))
   )
+  (wire (pts (xy 165.1 76.2) (xy 170.18 76.2))
+    (stroke (width 0) (type default))
+  )
   (wire (pts (xy 255.27 120.65) (xy 255.27 106.68))
     (stroke (width 0) (type default))
@@
     (stroke (width 0) (type default))
   )
+  (wire (pts (xy 134.62 55.88) (xy 134.62 73.66))
+    (stroke (width 0) (type default))
+  )
   (wire (pts (xy 19.05 88.9) (xy 19.05 58.42))
     (stroke (width 0) (type default))
@@
     (stroke (width 0) (type default))
   )
-  (wire (pts (xy 134.62 67.31) (xy 134.62 73.66))
-    (stroke (width 0) (type default))
-  )
   (wire (pts (xy 208.28 44.45) (xy 215.9 44.45))
     (stroke (width 0) (type default))
@@
     (stroke (width 0) (type default))
   )
-  (wire (pts (xy 161.29 72.39) (xy 161.29 67.31))
-    (stroke (width 0) (type default))
-  )
   (wire (pts (xy 54.61 55.88) (xy 54.61 58.42))
     (stroke (width 0) (type default))
@@
     (stroke (width 0) (type default))
   )
+  (wire (pts (xy 161.29 55.88) (xy 161.29 57.15))
+    (stroke (width 0) (type default))
+  )
   (wire (pts (xy 215.9 92.71) (xy 215.9 118.11))
     (stroke (width 0) (type default))
   )
-  (wire (pts (xy 161.29 80.01) (xy 161.29 83.82))
-    (stroke (width 0) (type default))
-  )
   (wire (pts (xy 38.1 69.85) (xy 72.39 69.85))
     (stroke (width 0) (type default))
@@
     (stroke (width 0) (type default))
   )
+  (wire (pts (xy 161.29 81.28) (xy 170.18 81.28))
+    (stroke (width 0) (type default))
+  )
   (wire (pts (xy 93.98 78.74) (xy 106.68 78.74))
     (stroke (width 0) (type default))
   )
+  (wire (pts (xy 161.29 83.82) (xy 170.18 83.82))
+    (stroke (width 0) (type default))
+  )
   (wire (pts (xy 115.57 104.14) (xy 115.57 97.79))
     (stroke (width 0) (type default))
@@
   )
   (wire (pts (xy 255.27 106.68) (xy 223.52 106.68))
+    (stroke (width 0) (type default))
+  )
+  (wire (pts (xy 170.18 83.82) (xy 170.18 81.28))
     (stroke (width 0) (type default))
   )
@@
     )
   )
-  (symbol (lib_id "Device:R") (at 161.29 76.2 0) (unit 1)
-    (in_bom yes) (on_board yes) (dnp no) (fields_autoplaced)
-    (property "Reference" "R31" (at 163.83 74.93 0)
-      (effects (font (size 1.27 1.27)) (justify left))
-    )
-    (property "Value" "100k" (at 163.83 77.47 0)
-      (effects (font (size 1.27 1.27)) (justify left))
-    )
-    (property "Footprint" "Resistor_THT:R_Axial_DIN0204_L3.6mm_D1.6mm_P5.08mm_Horizontal" (at 159.512 76.2 90)
-      (effects (font (size 1.27 1.27)) hide)
-    )
-    (property "Datasheet" "~" (at 161.29 76.2 0)
+  (symbol (lib_id "Device:R") (at 161.29 60.96 0) (unit 1)
+    (in_bom yes) (on_board yes) (dnp no) (fields_autoplaced)
+    (property "Reference" "R31" (at 163.83 59.69 0)
+      (effects (font (size 1.27 1.27)) (justify left))
+    )
+    (property "Value" "100k" (at 163.83 62.23 0)
+      (effects (font (size 1.27 1.27)) (justify left))
+    )
+    (property "Footprint" "Resistor_THT:R_Axial_DIN0204_L3.6mm_D1.6mm_P5.08mm_Horizontal" (at 159.512 60.96 90)
+      (effects (font (size 1.27 1.27)) hide)
+    )
+    (property "Datasheet" "~" (at 161.29 60.96 0)
       (effects (font (size 1.27 1.27)) hide)
     )
@@
     )
   )
+  (symbol (lib_id "Device:R_Potentiometer") (at 161.29 76.2 0) (unit 1)
+    (in_bom yes) (on_board yes) (dnp no) (fields_autoplaced)
+    (property "Reference" "RV1" (at 158.75 74.93 0)
+      (effects (font (size 1.27 1.27)) (justify right))
+    )
+    (property "Value" "R_Potentiometer" (at 158.75 77.47 0)
+      (effects (font (size 1.27 1.27)) (justify right))
+    )
+    (property "Footprint" "Potentiometer_THT:Potentiometer_Piher_PT-6-V_Vertical" (at 161.29 76.2 0)
+      (effects (font (size 1.27 1.27)) hide)
+    )
+    (property "Datasheet" "~" (at 161.29 76.2 0)
+      (effects (font (size 1.27 1.27)) hide)
+    )
+    (pin "1")
+    (pin "2")
+    (pin "3")
+    (instances
+      (project "TimerS"
+        (path "/78a5e9e2-666e-497f-a0eb-8939aa477525"
+          (reference "RV1") (unit 1)
+        )
+      )
+    )
+  )
   (symbol (lib_id "power:GND") (at 93.98 104.14 0) (unit 1)
     (in_bom yes) (on_board yes) (dnp no) (fields_autoplaced)
@@
     )
   )
-  (symbol (lib_id "power:+5V") (at 134.62 64.77 0) (unit 1)
-    (in_bom yes) (on_board yes) (dnp no) (fields_autoplaced)
-    (property "Reference" "#PWR039" (at 134.62 68.58 0)
-      (effects (font (size 1.27 1.27)) hide)
-    )
-    (property "Value" "+5V" (at 134.62 59.69 0)
-      (effects (font (size 1.27 1.27)))
-    )
-    (property "Footprint" "" (at 134.62 64.77 0)
-      (effects (font (size 1.27 1.27)) hide)
-    )
-    (property "Datasheet" "" (at 134.62 64.77 0)
-      (effects (font (size 1.27 1.27)) hide)
-    )
+  (symbol (lib_id "power:+5V") (at 134.62 50.8 0) (unit 1)
+    (in_bom yes) (on_board yes) (dnp no) (fields_autoplaced)
+    (property "Reference" "#PWR039" (at 134.62 54.61 0)
+      (effects (font (size 1.27 1.27)) hide)
+    )
+    (property "Value" "+5V" (at 134.62 45.72 0)
+      (effects (font (size 1.27 1.27)))
+    )
+    (property "Footprint" "" (at 134.62 50.8 0)
+      (effects (font (size 1.27 1.27)) hide)
+    )
+    (property "Datasheet" "" (at 134.62 50.8 0)
+      (effects (font (size 1.27 1.27)) hide)
+    )
